File: Eagle_Project/MCP960XL-L0X-RL0X_EVM_v1_Eagle_7.x.sch (EAGLE design)
At the start: 93 parts, among them J1 PCB_THERMOCOUPLE, J2 2X6 FEMALE, Q1 2N7002, Q2 2N7002, Q3 2N7002, Q4 S8050, Q5 S8050, Q6 S8050, Q7 S8050, Q8 S8050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

Commit message: 5st
Parts:
- removed U4: PCA9534, TS100:PCA9534
- added C11: 100nF/50V, microbuilder:CAP_CERAMIC0603
- added U2: MCP9601, TS100:MCP9601
- U3: value MCP9601 -> PCA9534; device TS100:MCP9601 -> TS100:PCA9534
Connections:
- net 3.3V: now also C11.P$1, U2.VDD
- net A0: now also U3.A0; no longer U4.A0
- net A1: now also U3.A1; no longer U4.A1
- net A2: now also U3.A2; no longer U4.A2
- net ADDR: now also U2.ADDR; no longer U3.ADDR
- net ALERT1: now also U2.ALERT1, U3.IO3; no longer U3.ALERT1, U4.IO3
- net ALERT2: now also U2.ALERT2, U3.IO2; no longer U3.ALERT2, U4.IO2
- net ALERT3: now also U2.ALERT3, U3.IO1; no longer U3.ALERT3, U4.IO1
- net ALERT4: now also U2.ALERT4, U3.IO0; no longer U3.ALERT4, U4.IO0
- net GND: now also C11.P$2, U2.GND@1, U2.GND@10, U2.GND@11, U2.GND@2, U2.GND@3, U2.GND@7, U2.GND@8, U2.GND@9, U3.VSS; no longer U3.GND@1, U3.GND@10, U3.GND@11, U3.GND@2, U3.GND@3, U3.GND@7, U3.GND@8, U3.GND@9, U4.VSS
- net INT_3V3: now also U3.!INT; no longer U4.!INT
- net N$20: now also U3.IO7; no longer U4.IO7
- net N$21: now also U3.IO6; no longer U4.IO6
- net OC_ALERT: now also U2.OC_ALERT, U3.IO4; no longer U3.OC_ALERT, U4.IO4
- net SCL_3V3: now also U2.SCL; no longer U4.SCL
- net SC_ALERT: now also U2.SC_ALERT, U3.IO5; no longer U3.SC_ALERT, U4.IO5
- net SDA_3V3: now also U2.SDA; no longer U4.SDA
- net VIN+: now also U2.VIN+; no longer U3.VIN+
- net VIN-: now also U2.VIN-; no longer U3.VIN-
- net VSENSE: now also U2.VSENSE; no longer U3.VSENSE
