File: Eagle_Project/MCP960XL-L0X-RL0X_EVM_v1_teardrops.brd (EAGLE design)
At the start: 33 x 71.1 mm, 95 parts, among them J1 PCB_THERMOCOUPLE, J2 2X6 FEMALE, Q1 2N7002, Q2 2N7002, Q3 2N7002, Q4 S8050, Q5 S8050, Q6 S8050, Q7 S8050, Q8 S8050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

Commit message: 5st
Parts:
- removed U4: PCA9534, TS100:HVQFN16_4X4_0.65MM
- added C11: 100nF/50V, microbuilder:0603
- added U2: MCP9601, TS100:VQFN20_5MM
- U3: value MCP9601 -> PCA9534; device TS100:VQFN20_5MM -> TS100:HVQFN16_4X4_0.65MM
- moved U3 8.76 mm to (0.00, -8.76)
Connections:
- removed net N$20: U4.10
- removed net N$21: U4.9
- removed net VDD: U4.14
- net 3.3V: now also C11.1, U2.8, U3.14; no longer U3.8
- net A0: now also U3.15; no longer U4.15
- net A1: now also U3.16; no longer U4.16
- net A2: now also U3.1; no longer U4.1
- net ADDR: now also U2.16; no longer U3.16
- net ALERT1: now also U2.11, U3.5; no longer U3.11, U4.5
- net ALERT2: now also U2.12, U3.4; no longer U3.12, U4.4
- net ALERT3: now also U2.14, U3.3; no longer U3.14, U4.3
- net ALERT4: now also U2.15, U3.2; no longer U3.15, U4.2
- net GND: now also C11.2, U2.1, U2.10, U2.13, U2.17, U2.18, U2.3, U2.5, U2.THRM, U3.6, U3.PAD; no longer U3.1, U3.10, U3.13, U3.17, U3.18, U3.3, U3.5, U3.THRM, U4.6, U4.PAD
- net INT_3V3: now also U3.11; no longer U4.11
- net OC_ALERT: now also U2.9, U3.7; no longer U3.9, U4.7
- net SCL_3V3: now also U2.19, U3.12; no longer U3.19, U4.12
- net SC_ALERT: now also U2.7, U3.8; no longer U3.7, U4.8
- net SDA_3V3: now also U2.20, U3.13; no longer U3.20, U4.13
- net VIN+: now also U2.2; no longer U3.2
- net VIN-: now also U2.4; no longer U3.4
- net VSENSE: now also U2.6; no longer U3.6
Routing:
- net 3.3V: track 114.6 -> 132.1 mm, vias 9 -> 11
- net GND: track 37.4 -> 52.4 mm, vias 107 -> 106
- net SC_ALERT: track 66.3 -> 79.3 mm
- net OC_ALERT: track 59.9 -> 70.5 mm
- net SDA_3V3: track 22.3 -> 32.2 mm
- net A2: track 25.0 -> 34.0 mm
- net ALERT2: track 52.5 -> 60.8 mm
- net ALERT1: track 58.5 -> 66.8 mm
- net ALERT4: track 53.2 -> 61.4 mm
- net ALERT3: track 58.0 -> 66.3 mm
- net A0: track 23.2 -> 31.5 mm
- net A1: track 23.1 -> 31.4 mm
- net ADDR: track 25.2 -> 30.7 mm
- net N$9: track 19.0 -> 23.7 mm
- net N$14: track 10.4 -> 15.1 mm
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Other:
- board text added: "JLCJLCJLCJLC"
