File: Eagle_Project/MCP960XL-L0X-RL0X_EVM_v1_teardrops.sch (EAGLE design)
At the start: 94 parts, among them J1 PCB_THERMOCOUPLE, J2 2X6 FEMALE, Q1 2N7002, Q2 2N7002, Q3 2N7002, Q4 S8050, Q5 S8050, Q6 S8050, Q7 S8050, Q8 S8050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

Commit message: 5st
Connections:
- removed net N$20: U3.IO7
- removed net N$21: U3.IO6
Changed lines of the file:
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@@
 <setting verticaltext="up"/>
 </settings>
-<grid distance="50" unitdist="mil" unit="mil" style="lines" multiple="1" display="yes" altdistance="25" altunitdist="mil" altunit="mil"/>
+<grid distance="0.1" unitdist="inch" unit="inch" style="lines" multiple="1" display="no" altdistance="0.01" altunitdist="inch" altunit="inch"/>
 <layers>
 <layer number="1" name="Top" color="4" fill="1" visible="no" active="no"/>
@@
 </segment>
 </net>
-<net name="N$20" class="0">
-<segment>
-<wire x1="482.6" y1="10.16" x2="485.14" y2="10.16" width="0.1524" layer="91"/>
-<pinref part="U3" gate="G$1" pin="IO7"/>
-</segment>
-</net>
-<net name="N$21" class="0">
-<segment>
-<wire x1="482.6" y1="7.62" x2="485.14" y2="7.62" width="0.1524" layer="91"/>
-<pinref part="U3" gate="G$1" pin="IO6"/>
-</segment>
-</net>
